Commit message: Added sensor node for kinetic and updated notes

File: robotiq_ft_sensor/urdf/robotiq_fts150.urdf.xacro (robot description, xacro)
@@ -18,5 +18,5 @@
                 <origin xyz="0 0 0" rpy="0 0 0" />
                 <geometry>
-                    <mesh filename="package://robotiq_force_torque_sensor/meshes/visual/robotiq_fts150.stl"/>
+                    <mesh filename="package://robotiq_ft_sensor/meshes/visual/robotiq_fts150.stl"/>
                 </geometry>
                 <material name="black"/>
@@ -25,5 +25,5 @@
                 <origin xyz="0 0 0" rpy="0 0 0" />
                 <geometry>
-                    <mesh filename="package://robotiq_force_torque_sensor/meshes/collision/robotiq_fts150.stl"/>
+                    <mesh filename="package://robotiq_ft_sensor/meshes/collision/robotiq_fts150.stl"/>
                 </geometry>
             </collision>
@@ -33,7 +33,7 @@
             <origin xyz="0 0 0.01625" rpy="0 0 0" />
             <parent link="${prefix}fts_robotside" />
-            <child link="${prefix}robotiq_force_torque_frame_id" />
+            <child link="${prefix}robotiq_ft_frame_id" />
         </joint>
-        <link name="${prefix}robotiq_force_torque_frame_id"/>
+        <link name="${prefix}robotiq_ft_frame_id"/>
         <!-- toolside frame -->
         <joint name="${prefix}toolside_joint" type="fixed" >
